Commit message: refactored state diagram and fully functioning again now, fixed precision reaching errors

File: scara_description/urdf/scara_core.xacro (robot description, xacro)
@@ -91,5 +91,5 @@
         <child link="carriage1_link" />
         <axis xyz="0 0 1" />
-        <limit lower="${carriage1_lz / 2}" upper="${column1_lz - carriage1_lz / 2}" effort="100.0"
+        <limit lower="${carriage1_lz / 2}" upper="${column1_lz - carriage1_lz / 2}" effort="500.0"
             velocity="0.1" />
     </joint>
@@ -116,5 +116,5 @@
         <child link="shoulder_link" />
         <axis xyz="0 0 1" />
-        <limit lower="${-pi * 0.9}" upper="${pi * 0.9}" effort="100" velocity="${pi}" />
+        <limit lower="${-pi * 0.9}" upper="${pi * 0.9}" effort="500" velocity="${pi}" />
     </joint>
     <!-- Elbow -->
@@ -140,5 +140,5 @@
         <child link="elbow_link" />
         <axis xyz="0 0 1" />
-        <limit lower="${-pi * 0.9}" upper="${pi * 0.9}" effort="100" velocity="${pi}" />
+        <limit lower="${-pi * 0.9}" upper="${pi * 0.9}" effort="500" velocity="${pi}" />
     </joint>
     <!-- End Effector -->
