Commit message: done with wafer simulation

File: scara_description/urdf/gz_plugins.xacro (robot description, xacro)
@@ -17,4 +17,5 @@
             <attach_topic>/vacuum/attach</attach_topic>
             <detach_topic>/vacuum/detach</detach_topic>
+            <detach_on_start>true</detach_on_start>
         </plugin>
     </gazebo>

File: scara_description/urdf/scara.ros2_control.xacro (robot description, xacro)
@@ -7,15 +7,21 @@
         <joint name="column1_carriage1_joint">
             <command_interface name="position" />
-            <state_interface name="position" />
+            <state_interface name="position">
+                <param name="initial_value">0.4</param>
+            </state_interface>
             <state_interface name="velocity" />
         </joint>
         <joint name="carriage1_shoulder_joint">
             <command_interface name="position" />
-            <state_interface name="position" />
+            <state_interface name="position">
+                <!-- <param name="initial_value">0.848230</param> -->
+            </state_interface>
             <state_interface name="velocity" />
         </joint>
         <joint name="shoulder_elbow_joint">
             <command_interface name="position" />
-            <state_interface name="position" />
+            <state_interface name="position">
+                <!-- <param name="initial_value">0.452389</param> -->
+            </state_interface>
             <state_interface name="velocity" />
         </joint>

File: scara_description/urdf/scara_core.xacro (robot description, xacro)
@@ -5,5 +5,5 @@
     <xacro:property name="base_ly" value="0.5" />
     <xacro:property name="base_lz" value="0.35" />
-    <xacro:property name="base_mass" value="16" />
+    <xacro:property name="base_mass" value="116" />
     <xacro:property name="column1_lx" value="0.2" />
     <xacro:property name="column1_ly" value="0.3" />
@@ -54,5 +54,5 @@
                 <box size="${column1_lx} ${column1_ly} ${column1_lz}" />
             </geometry>
-            <origin xyz="0 0 ${column1_lz / 2}" rpy="0 0 0" />
+            <origin xyz="0 0 ${column1_lz * 0.5}" rpy="0 0 0" />
             <material name="red" />
         </visual>
