Commit message: added inertials and collisionsto the urdf

File: litho_ws/src/stage_description/urdf/stage.urdf.xacro (robot description, xacro)
@@ -1,4 +1,5 @@
 <robot xmlns:xacro="http://www.ros.org/wiki/xacro" name="stage">
     <xacro:include filename="materials.xacro" />
+    <xacro:include filename="inertials.xacro" />
     <xacro:include filename="stage_core.xacro" />
     <xacro:include filename="stage.ros2_control.xacro" />

File: litho_ws/src/stage_description/urdf/stage_core.xacro (robot description, xacro)
@@ -4,21 +4,25 @@
     <xacro:property name="base_ly" value="0.2" />
     <xacro:property name="base_lz" value="0.02" />
+    <xacro:property name="base_mass" value="10" />
     <xacro:property name="x_stage_lx" value="0.15" />
     <xacro:property name="x_stage_ly" value="0.15" />
     <xacro:property name="x_stage_lz" value="0.015" />
+    <xacro:property name="x_stage_mass" value="0.1" />
+    <xacro:property name="x_stage_lower" value="0" />
+    <xacro:property name="x_stage_upper" value="0.025" />
     <xacro:property name="y_stage_lx" value="0.15" />
     <xacro:property name="y_stage_ly" value="0.15" />
     <xacro:property name="y_stage_lz" value="0.015" />
+    <xacro:property name="y_stage_mass" value="0.1" />
+    <xacro:property name="y_stage_lower" value="0" />
+    <xacro:property name="y_stage_upper" value="0.025" />
     <xacro:property name="z_stage_lx" value="0.1" />
     <xacro:property name="z_stage_ly" value="0.1" />
     <xacro:property name="z_stage_lz" value="0.01" />
-    <xacro:property name="x_stage_lower" value="0" />
-    <xacro:property name="x_stage_upper" value="0.025" />
-    <xacro:property name="y_stage_lower" value="0" />
-    <xacro:property name="y_stage_upper" value="0.025" />
+    <xacro:property name="z_stage_mass" value="0.05" />
     <xacro:property name="z_stage_lower" value="0" />
     <xacro:property name="z_stage_upper" value="0.025" />
-    <xacro:property name="stage_effort" value="100" />
-    <xacro:property name="stage_vel" value="0.0001" />
+    <xacro:property name="stage_effort" value="100" /> <!-- N/m -->
+    <xacro:property name="stage_vel" value="0.005" /> <!-- m/s -->
     <!-- Base -->
     <link name="base_footprint" />
@@ -31,4 +35,12 @@
             <material name="black" />
         </visual>
+        <collision>
+            <origin xyz="0 ${base_lz/2} 0" rpy="0 0 0" />
+            <geometry>
+                <box size="${base_lx} ${base_ly} ${base_lz}" />
+            </geometry>
+        </collision>
+        <xacro:box_inertial lx="${base_lx}" ly="${base_ly}" lz="${base_lz}" m="${base_mass}"
+            o_xyz="0 ${base_lz/2} 0" o_rpy="0 0 0" />
     </link>
     <joint name="footprint_base_joint" type="fixed">
@@ -46,4 +58,13 @@
             <material name="red" />
         </visual>
+        <collision>
+            <origin xyz="0 0 ${x_stage_lz/2}" rpy="0 0 0" />
+            <geometry>
+                <box size="${x_stage_lx} ${x_stage_ly} ${x_stage_lz}" />
+            </geometry>
+        </collision>
+        <xacro:box_inertial lx="${x_stage_lx}" ly="${x_stage_ly}" lz="${x_stage_lz}"
+            m="${x_stage_mass}"
+            o_xyz="0 0 ${x_stage_lz/2}" o_rpy="0 0 0" />
     </link>
     <joint name="base_x_stage_joint" type="prismatic">
@@ -64,4 +85,13 @@
             <material name="green" />
         </visual>
+        <collision>
+            <origin xyz="0 0 ${y_stage_lz/2}" rpy="0 0 0" />
+            <geometry>
+                <box size="${y_stage_lx} ${y_stage_ly} ${y_stage_lz}" />
+            </geometry>
+        </collision>
+        <xacro:box_inertial lx="${y_stage_lx}" ly="${y_stage_ly}" lz="${y_stage_lz}"
+            m="${y_stage_mass}"
+            o_xyz="0 0 ${y_stage_lz/2}" o_rpy="0 0 0" />
     </link>
     <joint name="x_y_stage_joint" type="prismatic">
@@ -82,4 +112,13 @@
             <material name="cyan" />
         </visual>
+        <collision>
+            <origin xyz="0 0 ${z_stage_lz/2}" rpy="0 0 0" />
+            <geometry>
+                <box size="${z_stage_lx} ${z_stage_ly} ${z_stage_lz}" />
+            </geometry>
+        </collision>
+        <xacro:box_inertial lx="${z_stage_lx}" ly="${z_stage_ly}" lz="${z_stage_lz}"
+            m="${z_stage_mass}"
+            o_xyz="0 0 ${z_stage_lz/2}" o_rpy="0 0 0" />
     </link>
     <joint name="y_z_stage_joint" type="prismatic">
