Commit message: fixed missing ros2_control joints

File: litho_ws/src/stage_description/urdf/stage.ros2_control.xacro (robot description, xacro)
@@ -16,4 +16,26 @@
             <state_interface name="effort" />
         </joint>
+        <joint name="x_y_stage_joint">
+            <command_interface name="position">
+                <!-- <param name="min">-15</param>
+            <param name="max">15</param> -->
+            </command_interface>
+            <state_interface name="position">
+                <!-- <param name="initial_value">1.0</param> -->
+            </state_interface>
+            <state_interface name="velocity" />
+            <state_interface name="effort" />
+        </joint>
+        <joint name="y_z_stage_joint">
+            <command_interface name="position">
+                <!-- <param name="min">-15</param>
+            <param name="max">15</param> -->
+            </command_interface>
+            <state_interface name="position">
+                <!-- <param name="initial_value">1.0</param> -->
+            </state_interface>
+            <state_interface name="velocity" />
+            <state_interface name="effort" />
+        </joint>
     </ros2_control>
 </robot>
